File: Project2.kicad_pcb (KiCad board)
At the start: 2 copper layers, 76 parts, among them J1 Header_8-Y1Y8, J10 CON-USB-MICROAB, J2 Header_8-X9X16, J3 Header_X17X24, J4 Header_8-P1P8, J5 MicroSD-PUSH_PULL, J6 Proj2Battery, J7 Header_P9P10, J8 Header_8-Y9Y16, J9 Header_8-X1X8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

Commit message: Almost the whole layout
Parts:
- moved C15 86.5 mm to (116.1, 116.4), turned to 90 degrees
- moved R15 85.3 mm to (117.9, 126.5)
- moved R16 81.6 mm to (117.9, 128.1), turned to 180 degrees
- moved R25 80.1 mm to (129.0, 101.5), turned to 270 degrees
- moved R24 79.6 mm to (130.4, 101.5), turned to 270 degrees
- moved R23 79.6 mm to (131.9, 101.5), turned to 270 degrees
- moved R2 79.6 mm to (123.0, 109.6), turned to 90 degrees
- moved R9 79.4 mm to (120.3, 126.5), turned to 180 degrees
- moved C20 78.8 mm to (118.4, 107.2), turned to 90 degrees
- moved R28 77.7 mm to (130.5, 99.2), turned to 270 degrees
- moved R29 77.0 mm to (129.0, 99.2), turned to 270 degrees
- moved R27 75.6 mm to (131.8, 99.2), turned to 270 degrees
- moved R4 75.5 mm to (124.3, 106.3)
- moved R3 75.3 mm to (121.0, 106.8), turned to 180 degrees
- moved L1 74.8 mm to (118.4, 121.2), turned to 180 degrees
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Connections:
- SW2 pad 2: (no net) -> Net-(R19-Pad2)
Other:
- net class Default: clearance 0.2 -> 0.1524; trace_width 0.25 -> 0.1524; via_dia 0.6 -> 0.5842; via_drill 0.4 -> 0.381
- rule trace_clearance: 0.2 -> 0.1524
- rule trace_min: 0.2 -> 0.1524
- rule via_min_drill: 0.3 -> 0.381
- rule via_min_size: 0.4 -> 0.5842

Commit message: ALL THE SIGNAL PINS
Parts:
- moved J1 39.7 mm to (140.5, 127.9), turned to 90 degrees
- moved J9 23.3 mm to (118.9, 136.8), turned to 0 degrees
- moved J2 20.3 mm to (110.0, 102.5)
- moved J3 16.6 mm to (110.0, 122.8), turned to 270 degrees
- moved U2 2.43 mm to (137.7, 105.0), turned to 0 degrees
- moved R4 0.28 mm to (124.0, 106.2), turned to 180 degrees
- turned C17 to 180 degrees
- turned R11 to 0 degrees
- turned R16 to 0 degrees
- turned R17 to 0 degrees
- turned R9 to 0 degrees
Connections:
- net USB_DM renamed USB_D_N
- net USB_DP renamed USB_D_P
- J4 pad 1: BOOT0_P1 -> BOOT0-P1
Routing:
- net RST#: track 0.03 -> 95.6 mm, vias 0 -> 1
- net SW_X17: track 0.00 -> 47.8 mm, vias 0 -> 2
- net X11: track 0.00 -> 46.0 mm, vias 0 -> 2
- net X12: track 0.00 -> 44.7 mm, vias 0 -> 2
- net BOOT0-P1: track 0.00 -> 39.3 mm, vias 0 -> 1
- net BLU_P2: track 0.00 -> 35.3 mm, vias 0 -> 2
- net SCL_X9: track 0.00 -> 34.1 mm, vias 0 -> 1
- net SDA_X10: track 0.00 -> 33.9 mm, vias 0 -> 1
- net YEL_P3: track 0.00 -> 32.6 mm, vias 0 -> 2
- net Y2: track 0.00 -> 29.9 mm
- net GRN_P4: track 0.00 -> 29.7 mm, vias 0 -> 3
- net RED_P5: track 0.00 -> 29.6 mm, vias 0 -> 3
- net Y3: track 0.00 -> 29.1 mm, vias 0 -> 2
- net Y1: track 0.00 -> 29.1 mm, vias 0 -> 1
- net Y4: track 0.00 -> 28.4 mm, vias 0 -> 2
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- added copper zone on In1.Cu, net 3V3
- added copper zone on In2.Cu, net GND
Other:
- board outline added: 38 x 48.7 mm
- copper layers 2 -> 4

Commit message: Finished Pass 1
Parts:
- moved J5 0.12 mm to (112.2, 104.7)
- turned J7 to 180 degrees
Routing:
- net GND: track 4.92 -> 80.6 mm, vias 2 -> 21
- net V+: track 5.53 -> 72.6 mm, vias 0 -> 4
- net 3V3: track 7.95 -> 63.7 mm, vias 0 -> 12
- net SDA_X10: track 33.9 -> 29.3 mm
- net GRN_P4: track 29.7 -> 28.5 mm
- net USB_ID: track 22.6 -> 21.4 mm
- net MMA_AVDD: track 18.6 -> 19.4 mm
- net Net-(C13-Pad1): track 8.96 -> 9.53 mm
- added copper zone on In1.Cu, net V+

Commit message: Finished
Connections:
- J4 pad 7: V+ -> GND
- J4 pad 8: GND -> V+
Routing:
- net V+: track 72.6 -> 37.5 mm
- net GND: track 80.6 -> 73.9 mm, vias 21 -> 22
- net Y9: track 21.9 -> 20.2 mm
- net Y10: track 22.2 -> 20.8 mm
- net 3V3: track 63.7 -> 62.7 mm
Other:
- board text added: "3V3"
- board text added: "A3V3"
- board text added: "BAT"
- board text added: "BLU"
- board text added: "BOOT0"
- board text added: "Eclectronics Project #2 Fall 2017 Coleman Ellis & Paige Pfenninger "Basically Just the PyBoard""
- board text added: "GND"
- board text added: "GRN"
- board text added: "RED"
- board text added: "RST"
- board text added: "V+"
- board text added: "VBU"
- board text added: "X1"
- board text added: "X10 SDA"
- board text added: "X11"
- board text added: "X12"
- board text added: "X17 SW"
- board text added: "X18"
- board text added: "X19"
- board text added: "X2"
- board text added: "X20"
- board text added: "X21"
- board text added: "X22"
- board text added: "X3"
- board text added: "X4"
- board text added: "X5"
- board text added: "X6"
- board text added: "X7"
- board text added: "X8"
- board text added: "X9 SCL"
- board text added: "Y1"
- board text added: "Y10"
- board text added: "Y11"
- board text added: "Y12"
- board text added: "Y2"
- board text added: "Y3"
- board text added: "Y4"
- board text added: "Y5"
- board text added: "Y6"
- board text added: "Y7"
- board text added: "Y8"
- board text added: "Y9"
- board text added: "YEL"
